File: pcb/ISA rev2 with remote/ISA card rev2.kicad_pcb (KiCad board)
At the start: 2 copper layers, 81.3 x 87.6 mm, 28 parts, among them J1 PCB_Finger_ISA_8bit, J2 OLED Header, J3 remote header, J4 OLED here, J5 Button Header, SW1 Up, SW2 Down, SW3 Select/Menu, U1 74LVC02, U2 74LVC245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

Commit message: more available 74LVC02 footprint; generate gbrs
Parts:
- U1: footprint Package_SO:SO-14_5.3x10.2mm_P1.27mm -> Package_SO:SO-14_3.9x8.65mm_P1.27mm
- moved U1 1.20 mm to (148.6, 132.1)
Routing:
- net GND: track 33.3 -> 43.3 mm, vias 10 -> 11
- net +3V3: track 190.0 -> 189.4 mm
- net /PA4: track 48.7 -> 49.3 mm

Commit message: rev4 board
Other:
- board text added: "18k"
Changed lines of the file:
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@@
     (effects (font (size 1 1) (thickness 0.15)))
   )
-  (gr_text "33k" (at 154.94 107.315 90) (layer "F.SilkS")
+  (gr_text "18k\n" (at 154.94 107.315 90) (layer "F.SilkS")
     (effects (font (size 1 1) (thickness 0.15)))
   )
