File: pcb/ISA rev5/ISA rev5.kicad_pcb (KiCad board)
At the start: 2 copper layers, 81.5 x 51.1 mm, 35 parts, among them J1 PCB_Finger_ISA_8bit, J2 OLED Header, J5 Button Header, U1 74LVC02, U2 74LVC11, U3 74LVC245, U4 74LVC245, U5 74LVC245, U6 Pico

Commit message: PCB rev 5.1
Parts:
- D1, D5: value 3.3V -> BAT54S; footprint modified ICs:TO-236AB_diode -> Package_TO_SOT_SMD:SOT-23_Handsoldering
Connections:
- D1 pad 1: /+5Vmon -> GND
- D1 pad 2: GND -> +3V3
- D1 pad 3: (no net) -> /+5Vmon
- D5 pad 1: /+12Vmon -> GND
- D5 pad 2: GND -> +3V3
- D5 pad 3: (no net) -> /+12Vmon
Routing:
- net +3V3: track 33.1 -> 39.0 mm, vias 7 -> 9
Other:
- board text added: "1 pPi = 1E-12 Pi"
- board text added: "5V 3V3 GND SDA SCL"
- board text added: "PicoPOST Dev Board v5.1 - 2022/11/13"
- board text added: "Up Down Select"
- board text removed: "PicoPOST Dev Board v5 - 2022/11/11"
