File: pcb/ISA rev5/ISA rev5.kicad_sch (KiCad schematic)
At the start: 40 parts, among them J1 PCB_Finger_ISA_8bit, J2 OLED Header, J3 remote header, J4 OLED here, J5 Button Header, SW1 Up, SW2 Down, SW3 Select/Menu, U1 74LVC02, U2 74LVC11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

Commit message: PCB rev 5.1
Parts:
- removed D1, D5: 3.3V, modified ICs:TO-236AB_diode, symbol Device:D_Zener
- added D1, D5: BAT54S, Package_TO_SOT_SMD:SOT-23_Handsoldering, symbol Diode:BAT54S
Connections:
- net +12Vmon: now also D5.3
- net +3V3: now also D1.2, D5.2
- net +5Vmon: now also D1.3
- net GND: now also D1.1, D5.1
Other:
- moved on the sheet: R1, R10, R11, R2
