File: pcb/ISA rev6/ISA rev6.kicad_pcb (KiCad board)
At the start: 2 copper layers, 81 x 68.3 mm, 37 parts, among them J1 PCB_Finger_ISA_8bit, J2 Remote Connector, J3 Power Select Jumper, U1 74LVC02, U2 74LVC11, U3 74LVC245, U4 74LVC245, U5 74LVC245, U6 Pico

Commit message: PCB rev 6 part deux
Routing:
- net +3V3: track 92.8 -> 93.4 mm
Other:
- board size 81 x 68.3 mm -> 82 x 68.3 mm
Changed lines of the file:
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@@
   (gr_line (start 153.924 65.278) (end 129.032 65.278) (layer "F.SilkS") (width 0.1524))
   (gr_arc (start 101.346 130.556) (mid 100.98679 130.40721) (end 100.838 130.048) (layer "Edge.Cuts") (width 0.0381))
+  (gr_line (start 182.88 121.158) (end 182.88 62.23) (layer "Edge.Cuts") (width 0.0381))
   (gr_line (start 100.838 130.048) (end 100.838 62.23) (layer "Edge.Cuts") (width 0.0381))
-  (gr_line (start 181.864 130.048) (end 181.864 62.23) (layer "Edge.Cuts") (width 0.0381))
+  (gr_line (start 181.864 121.158) (end 181.864 130.048) (layer "Edge.Cuts") (width 0.0381))
+  (gr_line (start 181.864 121.158) (end 182.88 121.158) (layer "Edge.Cuts") (width 0.0381))
   (gr_line (start 101.346 130.556) (end 181.356 130.556) (layer "Edge.Cuts") (width 0.0381))
+  (gr_line (start 182.88 62.23) (end 181.864 62.23) (layer "Edge.Cuts") (width 0.0381))
   (gr_line (start 181.864 62.23) (end 100.838 62.23) (layer "Edge.Cuts") (width 0.0381))
   (gr_arc (start 181.864 130.048) (mid 181.71521 130.40721) (end 181.356 130.556) (layer "Edge.Cuts") (width 0.0381))
@@
   (segment (start 156.148 119.888) (end 157.607 119.888) (width 0.127) (layer "F.Cu") (net 2))
   (segment (start 161.098 114.808) (end 161.098 116.078) (width 0.127) (layer "F.Cu") (net 2))
-  (segment (start 162.814 120.142) (end 163.304011 120.632011) (width 0.127) (layer "F.Cu") (net 2))
+  (segment (start 162.814 120.142) (end 163.304011 120.632011) (width 0.2) (layer "F.Cu") (net 2))
   (segment (start 102.992 114.3335) (end 102.992 111.384) (width 0.2) (layer "F.Cu") (net 2))
-  (segment (start 164.609989 120.632011) (end 165.1 120.142) (width 0.127) (layer "F.Cu") (net 2))
+  (segment (start 164.609989 120.632011) (end 165.1 120.142) (width 0.2) (layer "F.Cu") (net 2))
   (segment (start 102.992 111.384) (end 103.124 111.252) (width 0.2) (layer "F.Cu") (net 2))
-  (segment (start 162.814 119.253) (end 162.814 120.142) (width 0.127) (layer "F.Cu") (net 2))
+  (segment (start 162.814 119.253) (end 162.814 120.142) (width 0.2) (layer "F.Cu") (net 2))
   (segment (start 157.607 119.888) (end 157.734 119.761) (width 0.127) (layer "F.Cu") (net 2))
   (segment (start 165.1 120.142) (end 165.1 119.4135) (width 0.127) (layer "F.Cu") (net 2))
-  (segment (start 163.304011 120.632011) (end 164.609989 120.632011) (width 0.127) (layer "F.Cu") (net 2))
+  (segment (start 163.304011 120.632011) (end 164.609989 120.632011) (width 0.2) (layer "F.Cu") (net 2))
   (via (at 169.164 88.9) (size 0.6) (drill 0.3) (layers "F.Cu" "B.Cu") (free) (net 2))
   (via (at 104.394 98.806) (size 0.6) (drill 0.3) (layers "F.Cu" "B.Cu") (net 2))
@@
   (via (at 152.4 89.662) (size 0.6) (drill 0.3) (layers "F.Cu" "B.Cu") (free) (net 2))
   (segment (start 147.32 64.389) (end 147.447 64.262) (width 0.2) (layer "B.Cu") (net 2))
-  (segment (start 158.623 118.872) (end 159.004 119.253) (width 0.127) (layer "B.Cu") (net 2))
+  (segment (start 158.623 118.872) (end 159.004 119.253) (width 0.2) (layer "B.Cu") (net 2))
   (segment (start 147.32 67.945) (end 147.32 64.389) (width 0.2) (layer "B.Cu") (net 2))
   (segment (start 103.124 112.0575) (end 103.373 112.3065) (width 0.2) (layer "B.Cu") (net 2))
-  (segment (start 151.257 121.539) (end 155.956 121.539) (width 0.127) (layer "B.Cu") (net 2))
+  (segment (start 156.845 121.539) (end 157.734 120.65) (width 0.2) (layer "B.Cu") (net 2))
   (segment (start 164.7575 114.3885) (end 164.465 114.681) (width 0.2) (layer "B.Cu") (net 2))
   (segment (start 152.4 88.9) (end 169.164 88.9) (width 0.6) (layer "B.Cu") (net 2))
@@
   (segment (start 167.005 117.856) (end 167.005 117.174099) (width 0.2) (layer "B.Cu") (net 2))
   (segment (start 164.465 115.6796) (end 164.465 114.681) (width 0.2) (layer "B.Cu") (net 2))
-  (segment (start 159.004 119.253) (end 162.814 119.253) (width 0.127) (layer "B.Cu") (net 2))
+  (segment (start 159.004 119.253) (end 162.814 119.253) (width 0.2) (layer "B.Cu") (net 2))
   (segment (start 103.124 111.252) (end 103.124 112.0575) (width 0.2) (layer "B.Cu") (net 2))
-  (segment (start 103.373 97.785) (end 104.394 98.806) (width 0.127) (layer "B.Cu") (net 2))
-  (segment (start 155.956 121.539) (end 157.734 119.761) (width 0.127) (layer "B.Cu") (net 2))
+  (segment (start 157.734 120.65) (end 157.734 119.761) (width 0.2) (layer "B.Cu") (net 2))
+  (segment (start 103.373 97.785) (end 104.394 98.806) (width 0.2) (layer "B.Cu") (net 2))
   (segment (start 165.1 107.95) (end 168.91 107.95) (width 0.2) (layer "B.Cu") (net 2))
   (segment (start 152.4 90.424) (end 169.164 90.424) (width 0.6) (layer "B.Cu") (net 2))
-  (segment (start 158.623 118.872) (end 158.623 117.6405) (width 0.127) (layer "B.Cu") (net 2))
+  (segment (start 158.623 118.872) (end 158.623 117.6405) (width 0.2) (layer "B.Cu") (net 2))
   (segment (start 167.005 117.174099) (end 166.416901 116.586) (width 0.2) (layer "B.Cu") (net 2))
   (segment (start 169.164 89.662) (end 152.4 89.662) (width 0.6) (layer "B.Cu") (net 2))
   (segment (start 150.241 119.126) (end 150.241 117.5135) (width 0.127) (layer "B.Cu") (net 2))
   (segment (start 165.608 114.3885) (end 164.7575 114.3885) (width 0.2) (layer "B.Cu") (net 2))
-  (segment (start 157.734 119.761) (end 158.623 118.872) (width 0.127) (layer "B.Cu") (net 2))
+  (segment (start 157.734 119.761) (end 158.623 118.872) (width 0.2) (layer "B.Cu") (net 2))
   (segment (start 166.416901 116.586) (end 165.3714 116.586) (width 0.2) (layer "B.Cu") (net 2))
+  (segment (start 151.257 121.539) (end 156.845 121.539) (width 0.2) (layer "B.Cu") (net 2))
   (segment (start 103.373 97.4975) (end 103.373 97.785) (width 0.127) (layer "B.Cu") (net 2))
   (segment (start 153.405022 66.929) (end 158.242 71.765978) (width 0.127) (layer "F.Cu") (net 3))
@@
     (polygon
       (pts
-        (xy 181.991 122.682)
+        (xy 182.626 120.904)
+        (xy 181.991 120.904)
+        (xy 181.991 122.682001)
         (xy 100.965 122.682)
         (xy 100.965 62.357)
-        (xy 181.864 62.357)
+        (xy 182.626 62.357)
       )
     )
@@
     (polygon
       (pts
+        (xy 182.626 120.904)
+        (xy 182.0097 120.905534)
         (xy 181.991 122.682)
         (xy 100.965 122.682)
         (xy 100.965 62.357)
-        (xy 181.864 62.357)
+        (xy 182.626 62.357)
       )
     )

Commit message: final rev6 release
Routing:
- net +12V: track 103.2 -> 100.2 mm
