File: pcb/ISA rev7/remote.kicad_sch (KiCad schematic)
At the start: 20 parts, among them J1 Remote Connector, J2 Generic Connector, J3 PiOLED Connector, J4 Qwiic/STEMMA QT, J5 Config Jumpers, SW1 Up, SW2 Down, SW3 Select, SW4 Back, U1 AMS1117-3.3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

Commit message: Finalized rev7 including gerbers
Other:
- note added: "GND SDA SCL GND 5V IRQ GND"
- note removed: "GND IRQ 5V GND SCL SDA GND"
Changed lines of the file:
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@@
     (stroke (width 0) (type default) (color 0 0 0 0))
   )
-  (text "GND\nIRQ\n5V\nGND\nSCL\nSDA\nGND" (at 20.32 76.2 0)
+  (text "GND\nSDA\nSCL\nGND\n5V\nIRQ\nGND" (at 20.32 76.2 0)
     (effects (font (size 1.5 1.5)) (justify left bottom))
   )
