File: pcb/ISA rev8/ISA rev8.kicad_pcb (KiCad board)
At the start: 2 copper layers, 99.6 x 69.2 mm, 44 parts, among them J1 PCB_Finger_ISA_8bit, J2 Remote Cable, J3 Power Select Jumper, J4 Remote Hardmount Connector, J5 Buzzer, U1 74LVC02, U2 74LVC11, U3 74LVC245, U4 74LVC245, U5 74LVC245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

Commit message: rev8 PCB final?
Parts:
- added C2: 100n, Capacitor_SMD:C_1206_3216Metric_Pad1.33x1.80mm_HandSolder, B.Cu at (190.1, 71.9)
- J2: value Remote Cable -> Remote Connector
- U7: value 24LC00 -> 24LC01
Connections:
- R10 pad 1: +5V -> +3V3
Routing:
- net +5V: track 80.2 -> 64.5 mm, vias 2 -> 1
- net +3V3: track 42.6 -> 44.3 mm, vias 16 -> 17
Other:
- board text added: "24C0x"
- board text added: "Board rev 8 2024/01/21"
- board text removed: "Board rev 8 2024/01/15"
Changed lines of the file:
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@@
         (effects (font (size 1 1) (thickness 0.15)) (justify left))
     )
-    (fp_text value "Remote Cable" (at 0 0 90) (layer "F.SilkS")
+    (fp_text value "Remote Connector" (at 0 0 90) (layer "F.SilkS")
         (effects (font (size 1.27 1.27) (thickness 0.15)))
     )
@@
     (fp_line (start 1.6 0.8) (end -1.6 0.8)
       (stroke (width 0.1) (type solid)) (layer "F.Fab"))
-    (pad "1" smd roundrect (at -1.55 0 270) (size 1.3 1.75) (layers "F.Cu" "F.Paste" "F.Mask") (roundrect_rratio 0.192308)
+    (pad "1" smd roundrect (at -1.55 0 270) (size 1.3 1.75) (layers "F.Cu" "F.Paste" "F.Mask") (roundrect_rratio 0.1923076923)
       (net 12 "Net-(D5-A)") (pintype "passive"))
-    (pad "2" smd roundrect (at 1.55 0 270) (size 1.3 1.75) (layers "F.Cu" "F.Paste" "F.Mask") (roundrect_rratio 0.192308)
+    (pad "2" smd roundrect (at 1.55 0 270) (size 1.3 1.75) (layers "F.Cu" "F.Paste" "F.Mask") (roundrect_rratio 0.1923076923)
       (net 20 "Net-(J1--12V)") (pintype "passive"))
     (model "${KICAD6_3DMODEL_DIR}/Resistor_SMD.3dshapes/R_1206_3216Metric.wrl"
@@
   )
   (footprint "Capacitor_SMD:C_1206_3216Metric_Pad1.33x1.80mm_HandSolder" (layer "B.Cu")
+    (at 190.119 71.9205 90)
+    (descr "Capacitor SMD 1206 (3216 Metric), square (rectangular) end terminal, IPC_7351 nominal with elongated pad for handsoldering. (Body size source: IPC-SM-782 page 76, https://www.pcb-3d.com/wordpress/wp-content/uploads/ipc-sm-782a_amendment_1_and_2.pdf), generated with kicad-footprint-generator")
+    (tags "capacitor handsolder")
+    (property "Sheetfile" "ISA rev8.kicad_sch")
+    (property "Sheetname" "")
+    (property "ki_description" "Unpolarized capacitor, small symbol")
+    (property "ki_keywords" "capacitor cap")
+    (attr smd)
+    (fp_text reference "C2" (at 0.1655 -2.032 90) (layer "B.SilkS")
+        (effects (font (size 1 1) (thickness 0.15)) (justify mirror))
+    )
+    (fp_text value "100n" (at 0 -1.85 90) (layer "B.Fab")
+        (effects (font (size 1 1) (thickness 0.15)) (justify mirror))
+    )
+    (fp_text user "${REFERENCE}" (at 0 0 90) (layer "B.Fab")
+        (effects (font (size 0.8 0.8) (thickness 0.12)) (justify mirror))
+    )
+    (fp_line (start -0.711252 -0.91) (end 0.711252 -0.91)
+      (stroke (width 0.12) (type solid)) (layer "B.SilkS"))
+    (fp_line (start -0.711252 0.91) (end 0.711252 0.91)
+      (stroke (width 0.12) (type solid)) (layer "B.SilkS"))
+    (fp_line (start -2.48 -1.15) (end -2.48 1.15)
+      (stroke (width 0.05) (type solid)) (layer "B.CrtYd"))
+    (fp_line (start -2.48 1.15) (end 2.48 1.15)
+      (stroke (width 0.05) (type solid)) (layer "B.CrtYd"))
+    (fp_line (start 2.48 -1.15) (end -2.48 -1.15)
+      (stroke (width 0.05) (type solid)) (layer "B.CrtYd"))
+    (fp_line (start 2.48 1.15) (end 2.48 -1.15)
+      (stroke (width 0.05) (type solid)) (layer "B.CrtYd"))
+    (fp_line (start -1.6 -0.8) (end -1.6 0.8)
+      (stroke (width 0.1) (type solid)) (layer "B.Fab"))
+    (fp_line (start -1.6 0.8) (end 1.6 0.8)
+      (stroke (width 0.1) (type solid)) (layer "B.Fab"))
+    (fp_line (start 1.6 -0.8) (end -1.6 -0.8)
+      (stroke (width 0.1) (type solid)) (layer "B.Fab"))
+    (fp_line (start 1.6 0.8) (end 1.6 -0.8)
+      (stroke (width 0.1) (type solid)) (layer "B.Fab"))
+    (pad "1" smd roundrect (at -1.5625 0 90) (size 1.325 1.8) (layers "B.Cu" "B.Paste" "B.Mask") (roundrect_rratio 0.188679)
+      (net 66 "+5V") (pintype "passive"))
+    (pad "2" smd roundrect (at 1.5625 0 90) (size 1.325 1.8) (layers "B.Cu" "B.Paste" "B.Mask") (roundrect_rratio 0.188679)
+      (net 1 "GND") (pintype "passive"))
+    (model "${KICAD6_3DMODEL_DIR}/Capacitor_SMD.3dshapes/C_1206_3216Metric.wrl"
+      (offset (xyz 0 0 0))
+      (scale (xyz 1 1 1))
+      (rotate (xyz 0 0 0))
+    )
+  )
+  (footprint "Capacitor_SMD:C_1206_3216Metric_Pad1.33x1.80mm_HandSolder" (layer "B.Cu")
     (at 165.608 115.951 90)
     (descr "Capacitor SMD 1206 (3216 Metric), square (rectangular) end terminal, IPC_7351 nominal with elongated pad for handsoldering. (Body size source: IPC-SM-782 page 76, https://www.pcb-3d.com/wordpress/wp-content/uploads/ipc-sm-782a_amendment_1_and_2.pdf), generated with kicad-footprint-generator")
@@
         (effects (font (size 1 1) (thickness 0.15)) (justify mirror))
     )
-    (fp_text value "24LC00" (at 0 -3.4 90) (layer "B.Fab")
+    (fp_text value "24LC01" (at 0 -3.4 90) (layer "B.Fab")
         (effects (font (size 1 1) (thickness 0.15)) (justify mirror))
     )
@@
       (stroke (width 0.1) (type solid)) (layer "B.Fab"))
     (pad "1" smd roundrect (at -1.55 0 270) (size 1.3 1.75) (layers "B.Cu" "B.Paste" "B.Mask") (roundrect_rratio 0.1923076923)
-      (net 66 "+5V") (pintype "passive"))
+      (net 2 "+3V3") (pintype "passive"))
     (pad "2" smd roundrect (at 1.55 0 270) (size 1.3 1.75) (layers "B.Cu" "B.Paste" "B.Mask") (roundrect_rratio 0.1923076923)
       (net 101 "/revDetect") (pintype "passive"))
@@
     (effects (font (size 0.8128 0.8128) (thickness 0.1524)) (justify mirror))
   )
+  (gr_text "24C0x" (at 194.31 71.247) (layer "B.SilkS")
+    (effects (font (size 0.8128 0.8128) (thickness 0.1524)) (justify mirror))
+  )
   (gr_text "This side towards rear!" (at 198.628 71.628 -90) (layer "B.SilkS")
     (effects (font (size 0.8128 0.8128) (thickness 0.1524)) (justify mirror))
   )
-  (gr_text "Settings EEPROM" (at 185.928 71.374) (layer "B.SilkS")
+  (gr_text "Settings EEPROM" (at 186.055 68.58) (layer "B.SilkS")
     (effects (font (size 0.8128 0.8128) (thickness 0.1524)) (justify mirror))
   )
@@
     (effects (font (size 0.8128 0.8128) (thickness 0.1524)))
   )
-  (gr_text "Board rev 8\n2024/01/15" (at 124.587 95.3262) (layer "F.SilkS")
+  (gr_text "Board rev 8\n2024/01/21" (at 124.587 95.3262) (layer "F.SilkS")
     (effects (font (size 0.8128 0.8128) (thickness 0.1524)))
   )
@@
   (segment (start 165.1 120.142) (end 165.1 119.4135) (width 0.127) (layer "F.Cu") (net 2))
   (via (at 178.562 109.982) (size 0.6) (drill 0.3) (layers "F.Cu" "B.Cu") (free) (net 2))
+  (via (at 176.149 91.948) (size 0.6) (drill 0.3) (layers "F.Cu" "B.Cu") (net 2))
   (via (at 104.394 98.806) (size 0.6) (drill 0.3) (layers "F.Cu" "B.Cu") (net 2))
   (via (at 103.124 111.252) (size 0.6) (drill 0.3) (layers "F.Cu" "B.Cu") (net 2))
@@
   (segment (start 103.124 112.0575) (end 103.373 112.3065) (width 0.2) (layer "B.Cu") (net 2))
   (segment (start 156.845 121.539) (end 157.734 120.65) (width 0.2) (layer "B.Cu") (net 2))
+  (segment (start 176.276 93.446) (end 176.276 92.202) (width 0.127) (layer "B.Cu") (net 2))
   (segment (start 164.7575 114.3885) (end 164.465 114.681) (width 0.2) (layer "B.Cu") (net 2))
   (segment (start 178.562 109.982) (end 181.864 109.982) (width 0.4) (layer "B.Cu") (net 2))
@@
   (segment (start 164.465 115.6796) (end 164.465 114.681) (width 0.2) (layer "B.Cu") (net 2))
   (segment (start 159.004 119.253) (end 162.814 119.253) (width 0.2) (layer "B.Cu") (net 2))
+  (segment (start 176.149 91.948) (end 176.149 92.075) (width 0.127) (layer "B.Cu") (net 2))
   (segment (start 103.124 111.252) (end 103.124 112.0575) (width 0.2) (layer "B.Cu") (net 2))
   (segment (start 157.734 120.65) (end 157.734 119.761) (width 0.2) (layer "B.Cu") (net 2))
   (segment (start 103.373 97.785) (end 104.394 98.806) (width 0.2) (layer "B.Cu") (net 2))
+  (segment (start 176.276 92.202) (end 176.149 91.948) (width 0.127) (layer "B.Cu") (net 2))
   (segment (start 181.864 108.966) (end 178.562 108.966) (width 0.4) (layer "B.Cu") (net 2))
   (segment (start 158.623 118.872) (end 158.623 117.6405) (width 0.2) (layer "B.Cu") (net 2))
@@
   (segment (start 103.51 126.492) (end 103.51 116.2) (width 0.127) (layer "F.Cu") (net 65))
   (segment (start 193.802 77.252978) (end 193.802 91.666041) (width 0.2) (layer "F.Cu") (net 66))
-  (segment (start 193.352479 92.115562) (end 193.352479 92.143521) (width 0.127) (layer "F.Cu") (net 66))
   (segment (start 188.947022 72.398) (end 193.765022 77.216) (width 0.2) (layer "F.Cu") (net 66))
   (segment (start 193.802 91.666041) (end 193.352479 92.115562) (width 0.2) (layer "F.Cu") (net 66))
@@
   (segment (start 193.802 77.252978) (end 193.802 77.252978) (width 0.2) (layer "F.Cu") (net 66))
   (segment (start 191.492 112.334) (end 195.072 108.754) (width 0.4) (layer "F.Cu") (net 66))
-  (segment (start 193.352479 92.143521) (end 192.532 92.964) (width 0.127) (layer "F.Cu") (net 66))
-  (via (at 192.532 92.964) (size 0.6) (drill 0.3) (layers "F.Cu" "B.Cu") (net 66))
   (via (at 193.802 77.216) (size 0.6) (drill 0.3) (layers "F.Cu" "B.Cu") (net 66))
-  (segment (start 192.532 92.964) (end 192.05 93.446) (width 0.127) (layer "B.Cu") (net 66))
+  (segment (start 190.5 73.483) (end 191.977 73.483) (width 0.2) (layer "B.Cu") (net 66))
   (segment (start 192.278 75.692) (end 192.278 73.784) (width 0.127) (layer "B.Cu") (net 66))
   (segment (start 193.802 77.216) (end 192.278 75.692) (width 0.127) (layer "B.Cu") (net 66))
-  (segment (start 192.05 93.446) (end 176.276 93.446) (width 0.127) (layer "B.Cu") (net 66))
+  (segment (start 191.977 73.483) (end 192.278 73.784) (width 0.2) (layer "B.Cu") (net 66))
   (segment (start 136.17 75.972) (end 136.2075 76.0095) (width 0.127) (layer "F.Cu") (net 67))
   (segment (start 136.17 74.422) (end 136.17 75.972) (width 0.127) (layer "F.Cu") (net 67))
