File: pcb/ISA rev8/ISA rev8.kicad_sch (KiCad schematic)
At the start: 41 parts, among them J1 PCB_Finger_ISA_8bit, J2 Remote SATA Connector, J3 Power Select Jumper, J4 Remote Hardmount Connector, J5 Buzzer, U1 74LVC02, U2 74LVC11, U3 74LVC245, U4 74LVC245, U5 74LVC245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

Commit message: rev8 PCB final?
Parts:
- added C2: 100n, Capacitor_SMD:C_1206_3216Metric_Pad1.33x1.80mm_HandSolder, symbol Device:C_Small
- U7: value 24LC00 -> 24LC01
Connections:
- net +3V3: now also R10.1
- net +5V: now also C2.1; no longer R10.1
- net GND: now also C2.2
Other:
- note added: "Configuration EEPROM Higher capacity chips (eg. 24LC02, 04...) may be used"
- note added: "PC Speaker Passthrough"
- moved on the sheet: BZ1, J2, J4, J5, R10, R11, U7
