File: pcb/Pro rev1/Pro rev1.kicad_pcb (KiCad board)
At the start: 4 copper layers, 102.6 x 107.3 mm, 133 parts, among them J1 PCB_Finger_ISA_8bit, J2 USB C, J3 USB Select, J4 Remote SATA Connector, J5 MicroSD, J6 2350 SWD, J7 2040 SWD, J8 RJ45_Hanrun_HR911105A_Horizon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, SW2 P1_BS, U1 RP2350B-QFN80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

Commit message: updates and fixes to Pro rev1 PCB, possibly prod-ready?
Parts:
- added .: LOGO, project libraries:postcard_stamp, B.Cu at (110.0, 87.4)
- added C50: 100nF, Capacitor_SMD:C_0402_1005Metric, F.Cu at (170.8, 81.7)
- added C51: 100nF, Capacitor_SMD:C_0402_1005Metric, F.Cu at (169.8, 75.8)
- added SW4: 2040 Reset, Button_Switch_SMD:SW_SPST_TS-1088-xR020, F.Cu at (161.9, 95.5)
- C11, C12, C13, C14, C15, C43, C49, C7, C8, C9: footprint Capacitor_SMD:C_0201_0603Metric -> Capacitor_SMD:C_0402_1005Metric
- C2: footprint Resistor_SMD:R_0402_1005Metric -> Capacitor_SMD:C_0402_1005Metric
- C3, C31, C32, C5: footprint Resistor_SMD:R_0201_0603Metric -> Capacitor_SMD:C_0402_1005Metric
- D1: renamed from Main Status
- D6: value PMEG60T20ELR -> 3A SMAF; footprint Diode_SMD:Nexperia_CFP3_SOD-123W -> Diode_SMD:D_SMA
- D8: value red -> ISA Reset; footprint Diode_SMD:Nexperia_CFP3_SOD-123W -> Diode_SMD:D_0805_2012Metric
- D9: renamed from Eth Status
- FB1: footprint Diode_SMD:D_SOD-123 -> Inductor_SMD:L_0603_1608Metric
- L2: footprint Inductor_SMD:L_1812_4532Metric -> Inductor_SMD:L_APV_ANR4030
- R18: value 330 -> 470
- R19, R20, R21, R22: value 1000 -> 1k
- R23, R24: value 27R -> 22R
- R28, R3: footprint Resistor_SMD:R_0201_0603Metric -> Resistor_SMD:R_0402_1005Metric
- R38, R39: value 332R -> 470
- REF**: moved to B.Cu
- SW1: renamed from Eth Reset; footprint project libraries:SW_SPST_TS-1088-xR020 -> Button_Switch_SMD:SW_SPST_TS-1088-xR020
- SW2: footprint project libraries:SW_SPST_TS-1088-xR020 -> Button_Switch_SMD:SW_SPST_TS-1088-xR020
- SW3: renamed from RP2350 Reset; footprint project libraries:SW_SPST_TS-1088-xR020 -> Button_Switch_SMD:SW_SPST_TS-1088-xR020
- moved REF** 56.3 mm to (143.2, 54.2), turned to 180 degrees
- moved . 53.8 mm to (132.0, 111.9), turned to 180 degrees
- moved D8 13.2 mm to (118.4, 109.2), turned to 0 degrees
- moved . 7.22 mm to (112.4, 78.4)
- moved J7 4.03 mm to (159.3, 88.3)
- moved R36 1.81 mm to (171.1, 76.8)
- moved C7 1.28 mm to (154.2, 113.8)
- moved J8 0.86 mm to (182.5, 84.5)
- moved J4 0.74 mm to (194.3, 100.2)
- moved C15 0.72 mm to (139.2, 105.0), turned to 180 degrees
- moved J2 0.69 mm to (196.1, 48.5)
- moved D6 0.63 mm to (185.1, 54.3)
- moved C31 0.36 mm to (142.6, 87.8)
- moved C49 0.35 mm to (136.6, 117.3)
- moved C5 0.33 mm to (159.3, 109.7)
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Connections:
- C39 pad 1: +3V3 -> /RP2040/LAN_VDD
- FB1 pad 2: Net-(U14-VDD1A) -> /RP2040/LAN_VDD
- J8 pad 4: +3V3 -> /RP2040/LAN_VDD
- J8 pad 5: +3V3 -> /RP2040/LAN_VDD
- R37 pad 1: +3V3 -> /RP2040/LAN_VDD
- R40 pad 1: +3V3 -> /RP2040/LAN_VDD
- R41 pad 1: +3V3 -> /RP2040/LAN_VDD
- R42 pad 1: +3V3 -> /RP2040/LAN_VDD
- U13 pad 26: unconnected-(U13-RUN-Pad26) -> 2040_Reset
- U14 pad 1: Net-(U14-VDD1A) -> /RP2040/LAN_VDD
- U14 pad 19: Net-(U14-VDD1A) -> /RP2040/LAN_VDD
Routing:
- net 2040_Reset: track 0.00 -> 29.4 mm
- net /RP2040/LAN_VDD: track 0.00 -> 17.3 mm, vias 0 -> 7
- net Net-(U14-VDD1A): track 11.7 -> 0.00 mm, vias 2 -> 0
- net Net-(D8-A): track 1.65 -> 9.00 mm
- net P2_SWCLK: track 8.36 -> 12.5 mm
- net P2_SWDIO: track 12.7 -> 16.7 mm
- net VBUS: track 15.2 -> 11.3 mm
- net remote_SCL: track 68.5 -> 70.3 mm
- net remote_SDA: track 67.4 -> 69.0 mm
- net /RP2040/ETH_RXN: track 11.7 -> 13.1 mm
- net Net-(J1-RESET): track 78.0 -> 76.6 mm
- net GND: track 30.3 -> 31.5 mm, vias 72 -> 103
- net +3V3: track 139.1 -> 137.9 mm, vias 53 -> 46
- net /RP2040/ETH_RXP: track 17.8 -> 18.8 mm
- net Net-(J2-D--PadA7): track 9.07 -> 10.00 mm
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- added copper zone on In2.Cu, net /RP2040/LAN_VDD
Other:
- board text added: "-Douglas Adams"
- board text added: "1640 Riverside Drive Hill Valley, CA 91905"
- board text added: "Eth BOOTSEL"
- board text added: "Eth Reset"
- board text added: "Eth SWD"
- board text added: "Eth Status"
- board text added: "HW: Matthew Petry (fireTwoOneNine) SW: Enrico Zaghini (TheRealZago) Thanks to: Rigo (0xCats) PancakePuppy computerguy096 Deksor Ian Scott (polpo) The {dblquote}Retro Pico Hardware{dblquote} Discord Everyone who has contributed to TRW"
- board text added: "ISA Reset"
- board text added: "It's more than just a POST card... or a postcard."
- board text added: "Main BOOTSEL"
- board text added: "Main Reset"
- board text added: "Main SWD"
- board text added: "Main Status"
- board text added: "PCB rev 1 2025/08/23"
- board text added: "PicoPOST Pro"
- board text added: "This board requires 5V USB power!"
- board text added: "{dblquote}Technology is a word that describes something that doesn't work yet.{dblquote}"
- board text added: "❤"
- board text removed: "Board rev 1 2025/08/16"
- board text removed: "HW: Matthew Petry (fireTwoOneNine) SW: Enrico Zaghini (TheRealZago) Powered by TRW contributors Thanks: Rigo PancakePuppy computerguy096 Deksor Everyone in the Retro Pico Hardware Discord"
- board text removed: "RP2040 SWD"
- board text removed: "RP2350 SWD"
- board text removed: "The Ultimate ISA PC Diagnostic Tool"
