File: pcb/Pro rev1/pro-isa.kicad_sch (KiCad schematic)
At the start: 21 parts, among them J1 PCB_Finger_ISA_8bit, J2 USB C, J3 USB Select, J4 Remote SATA Connector, J5 MicroSD, J6 2350 SWD, J7 2040 SWD, U6 74LVC02

Commit message: updates and fixes to Pro rev1 PCB, possibly prod-ready?
Parts:
- D8: value red -> ISA Reset; footprint Diode_SMD:Nexperia_CFP3_SOD-123W -> Diode_SMD:D_0805_2012Metric
- R18: value 330 -> 470
- R19, R20, R21, R22: value 1000 -> 1k
- R23, R24: value 27R -> 22R
Changed lines of the file:
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@@
 	(title_block
 		(title "PicoPOST Pro")
-		(date "2025-08-12")
+		(date "2025-08-23")
 		(rev "1.0")
 		(company "The Retro Web")
@@
 			)
 		)
-		(property "Value" "27R"
+		(property "Value" "22R"
 			(at 134.62 35.3638 90)
 			(effects
@@
 			)
 		)
-		(property "Value" "1000"
+		(property "Value" "1k"
 			(at 80.01 123.19 90)
 			(effects
@@
 		(fields_autoplaced yes)
 		(property "Reference" "R18"
-			(at 46.99 43.8064 90)
+			(at 46.99 34.4889 90)
 			(effects
 				(font
@@
 			)
 		)
-		(property "Value" "330"
-			(at 46.99 41.2695 90)
+		(property "Value" "470"
+			(at 46.99 36.9132 90)
 			(effects
 				(font
@@
 			)
 		)
-		(property "Value" "red"
+		(property "Value" "ISA Reset"
 			(at 55.88 41.91 0)
 			(effects
@@
 			)
 		)
-		(property "Footprint" "Diode_SMD:Nexperia_CFP3_SOD-123W"
+		(property "Footprint" "Diode_SMD:D_0805_2012Metric"
 			(at 55.88 39.37 0)
 			(effects
@@
 			)
 		)
-		(property "Value" "1000"
+		(property "Value" "1k"
 			(at 80.01 118.11 90)
 			(effects
@@
 			)
 		)
-		(property "Value" "1000"
+		(property "Value" "1k"
 			(at 80.01 107.95 90)
 			(effects
@@
 			)
 		)
-		(property "Value" "1000"
+		(property "Value" "1k"
 			(at 80.01 113.03 90)
 			(effects
@@
 			)
 		)
-		(property "Value" "27R"
+		(property "Value" "22R"
 			(at 134.366 48.006 90)
 			(effects
