File: pcb/Pro rev1/pro-pwr-syslgc.kicad_sch (KiCad schematic)
At the start: 46 parts, among them SW1 P2_BS, SW2 P1_BS, U10 AP63203WU, U11 W25Q32JVSS, U12 24LC01, U2 74LVC245, U3 74LVC245, U4 MCP6002-T/SN, U5 74LVC245, U6 74LVC02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

Commit message: updates and fixes to Pro rev1 PCB, possibly prod-ready?
Parts:
- D6: value PMEG60T20ELR -> 3A SMAF; footprint Diode_SMD:Nexperia_CFP3_SOD-123W -> Diode_SMD:D_SMA
- L2: footprint Inductor_SMD:L_1812_4532Metric -> Inductor_SMD:L_APV_ANR4030
- SW1, SW2: footprint project libraries:SW_SPST_TS-1088-xR020 -> Button_Switch_SMD:SW_SPST_TS-1088-xR020
Changed lines of the file:
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@@
 			)
 		)
-		(property "Footprint" "Inductor_SMD:L_1812_4532Metric"
+		(property "Footprint" "Inductor_SMD:L_APV_ANR4030"
 			(at 254 133.35 0)
 			(effects
@@
 			)
 		)
-		(property "Value" "PMEG60T20ELR"
+		(property "Value" "3A SMAF"
 			(at 212.4075 135.4652 0)
 			(effects
@@
 			)
 		)
-		(property "Footprint" "Diode_SMD:Nexperia_CFP3_SOD-123W"
+		(property "Footprint" "Diode_SMD:D_SMA"
 			(at 212.09 133.985 0)
 			(effects
@@
 			)
 		)
-		(property "Footprint" "project libraries:SW_SPST_TS-1088-xR020"
+		(property "Footprint" "Button_Switch_SMD:SW_SPST_TS-1088-xR020"
 			(at 207.01 40.64 0)
 			(effects
@@
 			)
 		)
-		(property "Footprint" "project libraries:SW_SPST_TS-1088-xR020"
+		(property "Footprint" "Button_Switch_SMD:SW_SPST_TS-1088-xR020"
 			(at 123.19 40.64 0)
 			(effects
