File: pcb/Pro rev1/pro-rp2040.kicad_sch (KiCad schematic)
At the start: 38 parts, among them J8 RJ45_Hanrun_HR911105A_Horizon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, U13 RP2040, U14 LAN8720A, Y2 12MHz

Commit message: updates and fixes to Pro rev1 PCB, possibly prod-ready?
Parts:
- added C50, C51: 100nF, Capacitor_SMD:C_0402_1005Metric, symbol Device:C
- added SW4: 2040 Reset, Button_Switch_SMD:SW_SPST_TS-1088-xR020, symbol Switch:SW_Push
- C31, C32: footprint Resistor_SMD:R_0201_0603Metric -> Capacitor_SMD:C_0402_1005Metric
- FB1: footprint Diode_SMD:D_SOD-123 -> Inductor_SMD:L_0603_1608Metric
- R28: footprint Resistor_SMD:R_0201_0603Metric -> Resistor_SMD:R_0402_1005Metric
- R38, R39: value 332R -> 470
Connections:
- net +3V3: no longer C39.1, J8.4 (TCT), J8.5 (RCT), R37.1, R40.1, R41.1, R42.1
- net GND: now also C50.2, C51.2, SW4.2
- net 2040_Reset: now reaches U13.26 (RUN)
- net 2040_Reset: now also SW4.1
- net LAN_VDD: now reaches FB1.2, U14.1 (VDD2A), U14.19 (VDD1A)
- net LAN_VDD: now also C39.1, J8.4 (TCT), J8.5 (RCT), R37.1, R40.1, R41.1, R42.1, C50.1, C51.1
